File: Hardware/Custom_DUE/Arduino_DUE_X_V02d-2Layer.brd (EAGLE design)
At the start: 89 x 55.3 mm, 97 parts, among them IC1 LMV358IDGKR, IC10 74LVC1G125DCK, IC4 NCP1117ST33T3G -3V3, IC6 ATMEGA16U2-MU, J3 USB-MICRO B, T3 FDN340P, U1 ATSAM3X8EA-AU, U2 MCP2551, U3 LCD_DISPLAY, U4 MCP2551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

Commit message: Jaime
Parts:
- removed +12V_IN, GND_IN: TPPAD1-13, testpad:P1-13
- removed U$1: TLF1963TBATMA1, Dash parts:DPAK
- added +12, GND: TPPAD1-13, testpad:P1-13
- added AREF: TPB1,27, testpad:B1,27
- added U5: TLF1963TBATMA1, Dash parts:DPAK
- C1, C11, C2, C29, C3, C33: device rcl:SMC_B -> SmartPrj:C0805K
- Z3, Z4: device varistor:CT/CN0805 -> varistor:CT/CN0603
- moved RES 13.9 mm to (12.6, 39.1)
- moved SV3 11.0 mm to (4.06, 42.8)
- moved U3 6.76 mm to (16.6, 45.1)
- moved C33 2.06 mm to (38.0, 47.4), turned to 270 degrees
- moved C2 1.52 mm to (25.9, 42.7), turned to 270 degrees
- moved R25 1.40 mm to (79.1, 51.3), turned to 180 degrees
- moved C44 1.33 mm to (76.5, 30.4)
- moved R16 1.33 mm to (70.6, 24.6)
- moved R17 1.33 mm to (70.6, 21.5)
- moved C43 1.33 mm to (76.6, 23.1)
- moved IC1 1.33 mm to (70.4, 29.3)
- moved C11 0.96 mm to (35.1, 26.0), turned to 90 degrees
- moved C29 0.76 mm to (66.8, 22.0), turned to 270 degrees
- moved C3 0.76 mm to (45.2, 13.3), turned to 90 degrees
- moved C1 0.10 mm to (36.1, 13.0), turned to 0 degrees
- renumbered CANH_0 to CH0, CANH_1 to CH1, CANL_0 to CL0, CANL_1 to CL1
Connections:
- net N$20 renamed RES
- net +3V3: now also C1.2, C29.2; no longer C1.+, C29.+
- net +5V: now also U5.4; no longer U$1.4
- net AREF: now also AREF.TP
- net GND: now also C1.1, C11.1, C2.1, C29.1, C3.1, C33.1, GND.TP, U5.3, U5.6; no longer C1.-, C11.-, C2.-, C29.-, C3.-, C33.-, GND_IN.TP, U$1.3, U$1.6
- net N$13: now also +12.TP, U5.1, U5.2; no longer +12V_IN.TP, U$1.1, U$1.2
- net N$15: now also U5.5; no longer U$1.5
- net VDDANA: now also C3.2; no longer C3.+
- net VDDOUT: now also C11.2; no longer C11.+
- net VDDOUTMI: now also C2.2; no longer C2.+
- net VDDPLL: now also C33.2; no longer C33.+
Routing:
- net GND: track 480.7 -> 536.6 mm, vias 4 -> 22
- net +3V3: track 277.1 -> 246.2 mm, vias 10 -> 11
- net TX: track 108.8 -> 91.6 mm
- net N$21: track 0.00 -> 14.2 mm
- net N$19: track 0.00 -> 13.8 mm
- net N$18: track 0.00 -> 12.4 mm
- net N$22: track 0.00 -> 11.1 mm
- net RX: track 105.7 -> 100.5 mm, vias 4 -> 5
- net +5V: track 261.1 -> 257.4 mm, vias 13 -> 12
- net N$13: track 12.9 -> 16.6 mm
- net AREF: track 0.00 -> 3.22 mm
- net VDDPLL: track 11.8 -> 14.3 mm
- net VDDOUTMI: track 21.0 -> 22.9 mm
- net VDDOUT: track 114.2 -> 115.0 mm
- net RES: track 18.1 -> 18.8 mm
- added copper zone on layer 1, net GND
- added copper zone on layer 16, net GND
Other:
- board size 89 x 55.3 mm -> 83.5 x 55.2 mm
- board text added: "+"
- board text removed: "1"
- board text removed: "3V3"
- board text removed: "5V"
- board text removed: "ANALOG IN"
- board text removed: "AREF"
- board text removed: "Arduino"
- board text removed: "DIGITAL"
- board text removed: "DUE"
- board text removed: "GND"
- board text removed: "IOREF"
- board text removed: "ITALY"
- board text removed: "MADE IN"
- board text removed: "PWM"
- board text removed: "RESET"
- board text removed: "RX"
- board text removed: "RX0"
- board text removed: "RX1"
- board text removed: "RX3"
- board text removed: "SCL"
- board text removed: "SCL1"
- board text removed: "SDA"
- board text removed: "SDA1"
- board text removed: "TX"
- board text removed: "TX0"
- board text removed: "TX1"
- board text removed: "TX2"
- board text removed: "VIN"

Commit message: Jaime
Parts:
- moved L2 2.88 mm to (30.9, 34.0)
- moved R6 1.65 mm to (38.8, 41.5), turned to 270 degrees
- moved R5 1.35 mm to (35.1, 34.3)
- moved C36 0.52 mm to (13.5, 13.7)
- moved R27 0.33 mm to (68.1, 36.6)
- moved ERASE 0.25 mm to (23.4, 34.3)
Routing:
- net GND: track 536.6 -> 550.5 mm
- net +5V: track 257.4 -> 261.1 mm
- net N$12: track 8.96 -> 7.35 mm
- net AD2: track 24.9 -> 23.5 mm
- net N$11: track 4.54 -> 5.82 mm
- net VDDOUT: track 115.0 -> 116.0 mm
- net SS0/PWM10: track 6.78 -> 7.61 mm
- net N$1: track 6.29 -> 5.52 mm
- net D+: track 7.46 -> 6.82 mm
- net AD1: track 16.5 -> 17.0 mm
Other:
- board text added: "Digital Dash Rev.1, 03/28/2015 J.Rodriguez, N.Erickson R.Dass, S.Koppenhafer, C.Thueson"
