File: Hardware/Custom_DUE/Arduino_DUE_X_V02d-2Layer.sch (EAGLE design)
At the start: 96 parts, among them IC1 LMV358IDGKR, IC10 74LVC1G125DCK, IC4 NCP1117ST33T3G -3V3, IC6 ATMEGA16U2-MU, J3 USB-MICRO B, U1 ATSAM3X8EA-AU, U2 MCP2551, U4 MCP2551, Y1 12MHz KX-7 20pF, Y2 32.768Khz, Y4 16MHz KX-7 20pF

Commit message: Jaime
Parts:
- removed C20, C26: 10u, Dash parts:CPOL-US153CLV-0405
- removed R10, R3: 50, SmartPrj:R-EU_R0402
- removed R11, R12: 120, SmartPrj:R-EU_R0402
- removed R2: 3.5K, SmartPrj:R-EU_R0402
- removed U$3: LCD_DISPLAY, Dash parts:LCD_DISPLAY
- added C43, C44: 10u, Dash parts:CPOL-US153CLV-0405
- added JTAG: (no value), Arduino_Wifi_shield_v018_tG:PINHEAD_PINHD-2X5PASSO127
- added L, RX, TX: YELLOW, led:LEDCHIP-LED0805
- added ON: GREEN, led:LEDCHIP-LED0805
- added R17: 1K, SmartPrj:R-EU_R0805
- added R24, R26, R27: 50, SmartPrj:R-EU_R0805
- added R25, R28: 120, SmartPrj:R-EU_R0805
- added RN1, RN2: 100K, resistor-dil:4R-NCAT16
- added RN3: 1k, resistor-dil:4R-NCAY16
- added SV1, SV2, SV3: (no value), con-lsta:FE05-1
- added T1, T3, T4, T5, T8: TPB1,27, testpad:TPB1,27
- added T2: TPTP10R, testpad:TPTP10R
- added T6, T7: TPTP20SQ, testpad:TPTP20SQ
- added U3: LCD_DISPLAY, Dash parts:LCD_DISPLAY
- +12V_IN, CANH_0, CANH_1, CANL_0, CANL_1, GND_IN: value TPPAD1-20 -> TPPAD1-13; device testpad:TPPAD1-20 -> testpad:TPPAD1-13
- C10, C12, C13, C14, C15, C16, C17, C18, C19, C21, C22, C23, C24, C25, C28, C30, C32, C34, C36, C37, C38, C39, C4, C40, C5, C6, C7, C8, C9: device SmartPrj:C-EUC0402 -> SmartPrj:C-EUC0805
- JR1, R13, R14, R15, R18, R19, R20, R21, R22, R23, R4, R5, R6, R8, R9: device SmartPrj:R-EU_R0402 -> SmartPrj:R-EU_R0805
- R1: value 1K -> 0R; device SmartPrj:R-EU_R0402 -> SmartPrj:R-EU_R0805; SMD 1K, 1% -> (none)
- R16: value 50 -> 3.5K; device SmartPrj:R-EU_R0402 -> SmartPrj:R-EU_R0805; SMD (none) -> 3.5K, 1%
- R7: device SmartPrj:R-EU_R0603 -> SmartPrj:R-EU_R0805
- RES: value TPPAD1-20 -> TPB1,27; device testpad:TPPAD1-20 -> testpad:TPB1,27
- Z3, Z4: device varistor:VARISTORCN0603 -> varistor:VARISTORCN0805
Connections:
- removed net N$10: CANL_0.TP, R11.1, U4.CANL
- removed net N$6: R1.2, R2.1, U$1.VADJ
- removed net N$8: R16.2, R22.1, U4.VREF
- removed net N$9: CANH_0.TP, R11.2, U4.CANH
- new net AD11: SV3.3
- new net DAC0: SV2.2
- new net JTAG_RESET: JTAG.10, R1.1, RN1D.1
- new net L13: IC1A.-IN, IC1A.OUT, RN3C.2
- new net N$17: R22.1, R24.2, U4.VREF
- new net N$18: CANH_0.TP, R25.2, U4.CANH
- new net N$19: CANL_0.TP, R25.1, U4.CANL
- new net N$20: RES.TP, U3.RES
- new net N$21: CANH_1.TP, R28.2, U2.CANH
- new net N$22: CANL_1.TP, R28.1, U2.CANL
- new net N$54: RN3A.1, RX.A
- new net N$55: RN3B.1, TX.A
- net +3V3: now also JTAG.1, RN1C.2, RN1D.2, RN2B.1, RN2C.1, RN3A.2, RN3B.2, RN3D.2, SV3.4, T2.TP, T3.TP
- net +5V: now also C44.+, R16.2, R27.2, SV3.5, T4.TP, T8.TP, U3.+5; no longer C20.+, R10.2, R2.2, U$3.+5
- net AD0: now also SV2.5
- net AD1: now also SV2.4
- net AD2: now also SV2.3
- net DAC1: now also SV2.1
- net GND: now also C43.-, C44.-, JTAG.3, JTAG.5, JTAG.9, L.C, ON.C, R17.1, R24.1, R26.1, RN1A.1, RN1A.2, RN1B.1, RN1B.2, RN2A.1, RN2A.2, RN2D.1, RN2D.2, SV3.1, SV3.2, T5.TP, T6.TP, T7.TP, U3.GND; no longer C20.-, C26.-, R1.1, R16.1, R3.1, U$3.GND
- net JTAG_TCK: now also JTAG.4, RN2B.2
- net JTAG_TDI: now also JTAG.8, RN1C.1
- net JTAG_TDO: now also JTAG.6
- net JTAG_TMS: now also JTAG.2, RN2C.2
- net MASTER-RESET: now also R1.2, T1.TP
- net N$13: now also +12V_IN.TP, C43.+, U$1.EN, U$1.VIN; no longer CANH_1.TP, R12.2, U2.CANH
- net N$15: now also R16.1, R17.2, U$1.VADJ; no longer CANL_1.TP, R12.1, U2.CANL
- net N$16: now also R26.2, R27.1, U2.VREF; no longer RES.TP, U$3.RES
- net N$2: now also L.A, RN3C.1; no longer +12V_IN.TP, C26.+, U$1.EN, U$1.VIN
- net N$3: now also ON.A, RN3D.1; no longer R10.1, R3.2, U2.VREF
- net PWM13: now also IC1A.+IN
- net PWM2: now also SV1.5
- net PWM3: now also SV1.4
- net PWM5: now also SV1.2
- net PWM6: now also SV1.1
- net RX: now also U3.RX; no longer U$3.RX
- net RXL: now also RX.C
- net SS1/PWM4: now also SV1.3
- net TX: now also U3.TX; no longer U$3.TX
- net TXL: now also TX.C
Other:
- note added: "(ETH)"
- note added: "CONNECT"
- moved on the sheet: +12V_IN, BR1, C1, C10, C11, C12, C13, C14, C15, C16, C17, C18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

Commit message: jaime
Parts:
- removed FID1, FID2, FID3, FID4: FIDUCIALMOUNT, SmartPrj:FIDUCIALMOUNT
- removed JTAG: (no value), Arduino_Wifi_shield_v018_tG:PINHEAD_PINHD-2X5PASSO127
- removed L, RX, TX: YELLOW, led:LEDCHIP-LED0805
- removed ON: GREEN, led:LEDCHIP-LED0805
- removed R1: 0R, SmartPrj:R-EU_R0805
- removed RN1, RN2: 100K, resistor-dil:4R-NCAT16
- removed RN3: 1k, resistor-dil:4R-NCAY16
- removed SV1: (no value), con-lsta:FE05-1
- removed T1, T4, T5, T8: TPB1,27, testpad:TPB1,27
- removed T2: TPTP10R, testpad:TPTP10R
- removed T6, T7: TPTP20SQ, testpad:TPTP20SQ
- added ERASE: (no value), SmartPrj:MYSMD_PB157
- added R99: 10K, SmartPrj:R-EU_R0805
- T3: value TPB1,27 -> FDN340P; device testpad:TPB1,27 -> zetex:PMOSSOT23
Connections:
- net AD11 renamed NC
- removed net DAC0: SV2.2
- removed net JTAG_RESET: JTAG.10, R1.1, RN1D.1
- removed net L13: IC1A.-IN, IC1A.OUT, RN3C.2
- removed net N$2: L.A, RN3C.1
- removed net N$3: ON.A, RN3D.1
- removed net N$54: RN3A.1, RX.A
- removed net N$55: RN3B.1, TX.A
- net +3V3: now also ERASE.1, R99.2, T3.S; no longer JTAG.1, RN1C.2, RN1D.2, RN2B.1, RN2C.1, RN3A.2, RN3B.2, RN3D.2, T2.TP, T3.TP
- net +5V: no longer T4.TP, T8.TP
- net AD0: now also SV2.4; no longer SV2.5
- net AD1: now also SV2.3; no longer SV2.4
- net AD2: now also SV2.2; no longer SV2.3
- net AD3: now also SV2.1
- net DAC1: now also SV2.5; no longer SV2.1
- net ERASE_CMD: now also R99.1, T3.G
- net ERASE_S: now also ERASE.2, T3.D
- net GND: no longer JTAG.3, JTAG.5, JTAG.9, L.C, ON.C, RN1A.1, RN1A.2, RN1B.1, RN1B.2, RN2A.1, RN2A.2, RN2D.1, RN2D.2, T5.TP, T6.TP, T7.TP
- net JTAG_TCK: no longer JTAG.4, RN2B.2
- net JTAG_TDI: no longer JTAG.8, RN1C.1
- net JTAG_TDO: no longer JTAG.6
- net JTAG_TMS: no longer JTAG.2, RN2C.2
- net MASTER-RESET: no longer R1.2, T1.TP
- net PWM13: no longer IC1A.+IN
- net PWM2: no longer SV1.5
- net PWM3: no longer SV1.4
- net PWM5: no longer SV1.2
- net PWM6: no longer SV1.1
- net RXL: no longer RX.C
- net SS1/PWM4: no longer SV1.3
- net TXL: no longer TX.C
Other:
- note added: "ERASE"
- note removed: "CONNECT"
- moved on the sheet: +12V_IN, C29, C30, C43, C44, CANH_0, CANH_1, CANL_0, CANL_1, GND_IN, IC4, R16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

Commit message: Jaime
Parts:
- added AREF: TPB1,27, testpad:TPB1,27
- C1, C11, C2, C29, C3, C33: device rcl:CPOL-EUSMCB -> SmartPrj:C-EUC0805K
- Z3, Z4: device varistor:VARISTORCN0805 -> varistor:VARISTORCN0603
- renumbered +12V_IN to +12, CANH_0 to CH0, CANH_1 to CH1, CANL_0 to CL0, CANL_1 to CL1, GND_IN to GND, U$1 to U5
Connections:
- net N$20 renamed RES
- net +3V3: now also C1.2, C29.2; no longer C1.+, C29.+
- net AREF: now also AREF.TP
- net GND: now also C1.1, C11.1, C2.1, C29.1, C3.1, C33.1; no longer C1.-, C11.-, C2.-, C29.-, C3.-, C33.-
- net VDDANA: now also C3.2; no longer C3.+
- net VDDOUT: now also C11.2; no longer C11.+
- net VDDOUTMI: now also C2.2; no longer C2.+
- net VDDPLL: now also C33.2; no longer C33.+
