File: Hardware/FinalDesign/Arduino_DUE_X_V02d-2Layer.sch (EAGLE design)
At the start: 98 parts, among them IC1 LMV358IDGKR, IC10 74LVC1G125DCK, IC4 NCP1117ST33T3G -3V3, IC6 ATMEGA16U2-MU, J3 USB-MICRO B, T3 FDN340P, U1 ATSAM3X8EA-AU, U2 MCP2551, U3 LCD_DISPLAY, U4 MCP2551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

Commit message: Schematic cleanup for Jaime
Other:
- note added: "ATMEGA16"
- note added: "ATSAM3X"
- note added: "Bypass Caps"
- note added: "Headers"
- note added: "Power Supplies"
- note added: "Transceivers"
- moved on the sheet: AREF, BR1, C1, C10, C11, C12, C13, C14, C15, C16, C17, C18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
