File: Hardware/ATMEGA16u2Breakout/atmega16u2custom.brd (EAGLE design)
At the start: 61.9 x 45.7 mm, 58 parts, among them IC10 74LVC1G125DCK, J3 USB-MICRO B, U1 ATMEGA8U2AU

Commit message: atmega16u2 breakout board update
Parts:
- IC10: value 74LVC1G125DCK -> 74LVC1G125DBV; device 74xx-little-us:SC70-5 -> 74xx-little-us:SOT23-5
- Z3, Z4: device varistor:CT/CN0805 -> varistor:CT/CN0603
Routing:
- net GND: track 10.8 -> 15.1 mm, vias 5 -> 7
Changed lines of the file:
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@@
 <element name="D2" library="diode" package="MINIMELF" value="CD1206-S01575" x="55.245" y="31.115" rot="R90"/>
 <element name="F2" library="rcl" package="L1812" value="MF-MSMF050-2 500mA" x="7.62" y="16.51" rot="R270"/>
-<element name="IC10" library="74xx-little-us" package="SC70-5" value="74LVC1G125DCK" x="27.94" y="17.78" rot="R180"/>
+<element name="IC10" library="74xx-little-us" package="SOT23-5" value="74LVC1G125DBV" x="27.94" y="17.78" rot="R180"/>
 <element name="ICSP1" library="SmartPrj" package="2X03" value="3x2M" x="48.26" y="8.89" rot="R270"/>
 <element name="J3" library="SmartPrj" package="CON2_USB_MICRO_B_AT" value="USB-MICRO B" x="1.27" y="11.43" rot="R270"/>
@@
 <element name="TX1" library="led" package="CHIP-LED0805" value="YELLOW" x="33.655" y="13.335"/>
 <element name="U1" library="SparkFun-DigitalIC" package="TQFP32-08" value="ATMEGA8U2AU" x="35.56" y="27.94"/>
-<element name="Z3" library="varistor" package="CT/CN0805" value="CG0603MLC-05E" x="24.765" y="41.91"/>
-<element name="Z4" library="varistor" package="CT/CN0805" value="CG0603MLC-05E" x="8.255" y="8.89"/>
+<element name="Z3" library="varistor" package="CT/CN0603" value="CG0603MLC-05E" x="24.765" y="41.91"/>
+<element name="Z4" library="varistor" package="CT/CN0603" value="CG0603MLC-05E" x="8.255" y="8.89"/>
 <element name="TP1" library="testpad" package="B1,27" value="TPB1,27" x="26.67" y="31.75" smashed="yes">
 <attribute name="TP_SIGNAL_NAME" value="" x="26.035" y="29.845" size="1" layer="37"/>
@@
 <wire x1="35.96" y1="32.2326" x2="35.96" y2="37.465" width="0.4064" layer="1"/>
 <wire x1="35.96" y1="37.465" x2="36.83" y2="37.465" width="0.4064" layer="1"/>
-<polygon width="0.4064" layer="1">
+<polygon width="0.4064" layer="1" isolate="0.6096">
 <vertex x="0" y="0"/>
 <vertex x="61.595" y="0"/>
@@
 <vertex x="0" y="45.72"/>
 </polygon>
-<polygon width="0.4064" layer="16">
+<polygon width="0.4064" layer="16" isolate="0.6096">
 <vertex x="0" y="0"/>
 <vertex x="61.595" y="0"/>
@@
 <via x="29.21" y="33.655" extent="1-16" drill="0.6"/>
 <via x="21.59" y="41.91" extent="1-16" drill="0.6"/>
+<via x="24.765" y="17.78" extent="1-16" drill="0.6" shape="octagon"/>
+<wire x1="26.99" y1="19.07" x2="26.67" y2="18.63" width="0.4064" layer="1"/>
+<wire x1="26.67" y1="18.63" x2="26.67" y2="18.415" width="0.4064" layer="1"/>
+<wire x1="26.67" y1="18.415" x2="24.765" y2="18.415" width="0.4064" layer="1"/>
+<wire x1="24.765" y1="18.415" x2="24.765" y2="17.78" width="0.4064" layer="1"/>
+<via x="27.305" y="7.62" extent="1-16" drill="0.6" shape="octagon"/>
+<wire x1="3.9624" y1="9.0678" x2="3.9624" y2="10.1092" width="0.4064" layer="1"/>
 </signal>
 <signal name="+3V3">
@@
 <contactref element="C37" pad="1"/>
 <wire x1="27.52" y1="13.335" x2="28.59" y2="13.335" width="0.4064" layer="1"/>
-<wire x1="28.59" y1="13.335" x2="28.59" y2="16.93" width="0.4064" layer="1"/>
+<wire x1="28.59" y1="13.335" x2="28.89" y2="16.48" width="0.4064" layer="1"/>
 </signal>
 <signal name="USBVCC">
@@
 <wire x1="31.75" y1="20.955" x2="30.48" y2="20.955" width="0.4064" layer="1"/>
 <wire x1="30.48" y1="20.955" x2="28.59" y2="20.955" width="0.4064" layer="1"/>
-<wire x1="28.59" y1="20.955" x2="28.59" y2="18.63" width="0.4064" layer="1"/>
-<wire x1="27.94" y1="18.63" x2="28.59" y2="18.63" width="0.4064" layer="1"/>
+<wire x1="28.59" y1="20.955" x2="28.89" y2="19.07" width="0.4064" layer="1"/>
+<wire x1="27.94" y1="19.07" x2="28.89" y2="19.07" width="0.4064" layer="1"/>
 </signal>
 <signal name="N$4">
@@
 <contactref element="J3" pad="P2"/>
 <contactref element="R19" pad="2"/>
-<wire x1="30.265" y1="41.91" x2="25.865" y2="41.91" width="0.4064" layer="1"/>
+<wire x1="30.265" y1="41.91" x2="25.765" y2="41.91" width="0.4064" layer="1"/>
 <wire x1="3.9624" y1="12.0904" x2="11.43" y2="12.0904" width="0.4064" layer="1"/>
 <wire x1="11.43" y1="12.0904" x2="11.43" y2="13.97" width="0.4064" layer="1"/>
-<wire x1="25.865" y1="41.91" x2="26.035" y2="41.275" width="0.4064" layer="1"/>
-<wire x1="26.035" y1="41.275" x2="26.035" y2="40.005" width="0.4064" layer="1"/>
-<via x="26.035" y="40.005" extent="1-16" drill="0.6" shape="square"/>
-<wire x1="26.035" y1="40.005" x2="10.16" y2="40.005" width="0.4064" layer="16"/>
+<wire x1="25.765" y1="41.91" x2="26.035" y2="41.275" width="0.4064" layer="1"/>
+<wire x1="26.035" y1="41.275" x2="26.035" y2="40.64" width="0.4064" layer="1"/>
+<via x="26.035" y="40.64" extent="1-16" drill="0.6" shape="square"/>
+<wire x1="26.035" y1="40.64" x2="10.16" y2="40.005" width="0.4064" layer="16"/>
 <via x="11.43" y="13.97" extent="1-16" drill="0.6" shape="square"/>
 <wire x1="11.43" y1="13.97" x2="10.16" y2="13.97" width="0.4064" layer="16"/>
@@
 <contactref element="R20" pad="2"/>
 <wire x1="3.9624" y1="11.43" x2="9.355" y2="11.43" width="0.4064" layer="1"/>
-<wire x1="9.355" y1="11.43" x2="9.355" y2="8.89" width="0.4064" layer="1"/>
+<wire x1="9.355" y1="11.43" x2="9.255" y2="8.89" width="0.4064" layer="1"/>
 <via x="8.255" y="41.275" extent="1-16" drill="0.6" shape="square"/>
 <wire x1="8.255" y1="41.275" x2="8.255" y2="39.37" width="0.4064" layer="1"/>
